Commit message: rear axle controller

File: src/FirstTry_URDF/urdf/FirstTry_URDF.urdf (robot description, URDF)
Before this commit: robot FirstTry_URDF, 6 links, 5 joints
Links:
- added link dummy_link
- link chasis: mass 50.0082010252954 -> 10.00
- link left_castor: mass 1.31069724129228 -> 0.5
- link left_wheel: mass 2.31666659443376 -> 0.5
- link rear_axle: mass 5.50851834676472 -> 0.5
- link right_castor: mass 1.31069724129228 -> 0.5
- link right_wheel: mass 2.31666659443376 -> 0.5
Joints:
- added joint dummy_joint: type fixed, parent dummy_link, child chasis, origin xyz=0 0 0 rpy=0 0 0, axis 0 0 0
- joint rear_axle_joint: limit lower=0 upper=0 effort=0 velocity=0 -> lower=-1000000 upper=1000000 effort=10 velocity=100

Commit message: all controllers added
bot running yaayyy!

File: src/FirstTry_URDF/urdf/FirstTry_URDF.urdf (robot description, URDF)
Before this commit: robot FirstTry_URDF, 7 links, 6 joints
Joints:
- joint left_castor_joint: limit lower=0 upper=0 effort=0 velocity=0 -> lower=-1000000 upper=1000000 effort=10 velocity=100
- joint left_wheel_joint: limit lower=0 upper=0 effort=0 velocity=0 -> lower=-1000000 upper=1000000 effort=10 velocity=100
- joint right_castor_joint: limit lower=0 upper=0 effort=0 velocity=0 -> lower=-1000000 upper=1000000 effort=10 velocity=100
- joint right_wheel_joint: limit lower=0 upper=0 effort=0 velocity=0 -> lower=-1000000 upper=1000000 effort=10 velocity=100
