Commit message: changed world

File: src/FirstTry_URDF/urdf/ydlidar.urdf (robot description, URDF)
Before this commit: robot ydlidar, 2 links, 1 joints
Links:
- link base_laser: geometry collision mesh filename=package://FirstTry_URDF/meshes/ydlidar.dae; visual mesh filename=package://FirstTry_URDF/meshes/ydlidar.dae
- link laser_frame: geometry collision mesh filename=package://FirstTry_URDF/meshes/ydlidar.dae; visual mesh filename=package://FirstTry_URDF/meshes/ydlidar.dae

File: src/FirstTry_URDF/xacro/my_robot_integration.urdf.xacro (robot description, xacro)
@@ -17,4 +17,46 @@
 		</plugin>
 	</gazebo>
+<gazebo reference="base_laser">
+		<!-- <gravity>true</gravity> -->
+		<!-- Gazebo has fixed set of Sensors types. Check them out here <> -->
+		<sensor name="laser" type="ray">
+			<!-- Add in your sensor characteristics -->
+			<pose> 0 0 0 0 0 0 </pose>
+			<visualise>true</visualise>
+			<update_rate>40</update_rate>
+			<!-- <always_on>true</always_on> -->
+			<ray>
+				<scan>
+					<horizontal>
+						<samples>720</samples>
+						<resolution>1</resolution>
+						<min_angle>-1.570796</min_angle>
+              			<max_angle>1.570796</max_angle>
+              		</horizontal>
+              	</scan>
+              	<range>
+              		<min>0.10</min>
+              		<max>30.0</max>
+              		<resolution>0.01</resolution>
+              	</range>
+              	<noise>
+              		<type>gaussian</type>
+              		<mean>0.0</mean>
+              		<stddev>0.01</stddev>
+              	</noise>
+            </ray>
+            <plugin name="gazebo_ros_head_hokuyo_controller" filename="libgazebo_ros_laser.so">
+            	<!-- Use topic name as /my_robot/scan -->
+				<topicName>/castorbot/scan</topicName>
+				<frameName>laser_frame</frameName>
+			</plugin>
+		</sensor>
+	</gazebo>
 <!-- Create a joint between your robot and sensor -->
+  <joint name="lidar_joint" type="fixed">
+    <origin rpy="0 0 0" xyz="0 0 0.2"/>
+    <parent link="chasis"/>
+    <child link="base_laser"/>
+    <axis xyz="0 0 0"/>
+  </joint>
 </robot>
