Commit message: Added grasper

File: src/project2/door_u/urdf/door_u.urdf (robot description, URDF)
Before this commit: robot door_u, 2 links, 1 joints
Links:
- link door: mass 2 -> 0.01

Commit message: Make the final changes

File: src/project2/door_u/urdf/door_u.urdf (robot description, URDF)
Before this commit: robot door_u, 2 links, 1 joints
Links:
- link door_base: mass 10 -> 1000
